Commit message: Add elbow links and joints.

File: urdf/elbow.urdf.xacro (robot description, xacro)
@@ -1,18 +1,57 @@
 <?xml version='1.0' encoding='UTF-8'?>
 <robot xmlns:xacro='http://www.ros.org/wiki/xacro'>
-<xacro:macro name='el_link' params='name'>
+<xacro:macro name='el_link' params='name *shape reflectx:=1 roll:=0 pitch:=0 yaw:=0 x:=0 y:=0 z:=0 material:=blue'>
   <link name='elbow${name}'>
-    <!-- <visual> -->
-      <!-- <geometry> -->
-      <!-- </geometry> -->
-    <!-- </visual> -->
+    <visual>
+      <geometry>
+        <xacro:insert_block name='shape'/>
+      </geometry>
+      <origin rpy='${roll} ${pitch} ${yaw}' xyz='${x*reflectx} ${y} ${z}'/>
+      <material name='${material}'/>
+    </visual>
+    <collision>
+      <geometry>
+        <xacro:insert_block name='shape'/>
+      </geometry>
+      <origin rpy='${roll} ${pitch} ${yaw}' xyz='${x} ${y} ${z}'/>
+    </collision>
   </link>
 </xacro:macro>
-<xacro:macro name='el_joint' params='parent child type:=fixed'>
+<xacro:macro name='el_joint' params='parent child type:=fixed roll:=0 pitch:=0 yaw:=0 x:=0 y:=0 z:=0 axisx:=0 axisy:=0 axisz:=0'>
   <joint name='el${parent}_el${child}' type='${type}'>
     <parent link='elbow${parent}'/>
     <child link='elbow${child}'/>
-    <origin rpy='0 0 0' xyz='0 0 0'/>
-    <limit effort='300.0' lower='-0.5' upper='0.5' velocity='5.0'/>
+    <origin rpy='${roll} ${pitch} ${yaw}' xyz='${x} ${y} ${z}'/>
+    <limit effort='50.0' lower='-0.1' upper='0.1' velocity='5.0'/>
+    <axis xyz='${axisx} ${axisy} ${axisz}'/>
+  </joint>
+</xacro:macro>
+<xacro:macro name='el_refl_joint' params='parent child mimic type:=fixed roll:=0 pitch:=0 yaw:=0 x:=0 y:=0 z:=0 axisx:=0 axisy:=0 axisz:=0'>
+  <joint name='el${parent}_el${child}' type='${type}'>
+    <parent link='elbow${parent}'/>
+    <child link='elbow${child}'/>
+    <origin rpy='${roll} ${pitch} ${yaw}' xyz='${x} ${y} ${z}'/>
+    <limit effort='50.0' lower='-0.1' upper='0.1' velocity='5.0'/>
+    <axis xyz='${axisx} ${axisy} ${axisz}'/>
+    <mimic joint='${mimic}'/>
+  </joint>
+</xacro:macro>
+<xacro:macro name='el_cust_joint' params='parent child name type:=fixed roll:=0 pitch:=0 yaw:=0 x:=0 y:=0 z:=0 axisx:=0 axisy:=0 axisz:=0'>
+  <joint name='${name}' type='${type}'>
+    <parent link='${parent}'/>
+    <child link='${child}'/>
+    <origin rpy='${roll} ${pitch} ${yaw}' xyz='${x} ${y} ${z}'/>
+    <limit effort='50.0' lower='-0.1' upper='0.1' velocity='5.0'/>
+    <axis xyz='${axisx} ${axisy} ${axisz}'/>
+  </joint>
+</xacro:macro>
+<xacro:macro name='el_cust_refl_joint' params='parent child name mimic type:=fixed roll:=0 pitch:=0 yaw:=0 x:=0 y:=0 z:=0 axisx:=0 axisy:=0 axisz:=0'>
+  <joint name='${name}' type='${type}'>
+    <parent link='${parent}'/>
+    <child link='${child}'/>
+    <origin rpy='${roll} ${pitch} ${yaw}' xyz='${x} ${y} ${z}'/>
+    <limit effort='50.0' lower='-0.1' upper='0.1' velocity='5.0'/>
+    <axis xyz='${axisx} ${axisy} ${axisz}'/>
+    <mimic joint='${mimic}'/>
   </joint>
 </xacro:macro>

File: urdf/rehab.urdf.xacro (robot description, xacro)
@@ -6,5 +6,9 @@
 <xacro:include filename='$(find rehab)/urdf/hand.urdf.xacro'/>
 <!-- Link dimensions -->
-<xacro:property name='baselen' value='0.8'/>
+<!-- Base pole dimensions -->
+<xacro:property name='polelen' value='2'/>
+<xacro:property name='polerad' value='0.12'/>
+<!-- Connecting base plate dimensions -->
+<xacro:property name='basepllen' value='1.1'/>
 <xacro:property name='basethick' value='0.05'/>
 <xacro:property name='sh1len' value='0.25'/>
@@ -18,5 +22,5 @@
 <xacro:property name='mot2rad' value='0.1'/>
 <xacro:property name='mot2len' value='0.2'/>
-<!-- Second prismatic dimensions -->
+<!-- Third prismatic dimensions -->
 <xacro:property name='prism3len' value='0.25'/>
 <!-- Link for third motor -->
@@ -28,5 +32,33 @@
 <xacro:property name='shintrad' value='0.2'/>
 <xacro:property name='shintthick' value='0.05'/>
+<!-- Elbow dimensions -->
+<!-- Symmetric elbow connecting links dimensions -->
+<xacro:property name='elcon1len' value='0.35'/>
+<xacro:property name='elcon1width' value='0.1'/>
+<xacro:property name='elcon1thick' value='0.04'/>
+<!-- Symmetric elbow to forearm connecting links dimensions -->
+<xacro:property name='elcon2len' value='0.35'/>
+<xacro:property name='elcon2width' value='0.08'/>
+<xacro:property name='elcon2thick' value='0.04'/>
+<!-- Fourth motor dimensions -->
+<xacro:property name='mot4rad' value='0.04'/>
+<xacro:property name='mot4len' value='0.1'/>
+<!-- Fourth prismatic dimensions -->
+<xacro:property name='prism4len' value='0.1'/>
+<xacro:property name='prism4width' value='0.05'/>
+<xacro:property name='prism4thick' value='0.025'/>
+<!-- Elbow interface dimensions -->
+<xacro:property name='elintrad' value='0.16'/>
+<xacro:property name='elintthick' value='0.03'/>
+<!-- Fifth motor dimensions -->
+<xacro:property name='mot5rad' value='0.04'/>
+<xacro:property name='mot5len' value='0.1'/>
 <!-- Material colors -->
+<material name='red'>
+  <color rgba='0.8 0 0 1'/>
+</material>
+<material name='green'>
+  <color rgba='0 0.8 0 1'/>
+</material>
 <material name='blue'>
   <color rgba='0 0 0.8 1'/>
@@ -45,19 +77,19 @@
   <visual>
     <geometry>
-      <box size='${baselen} 0.3 ${basethick}'/>
+      <cylinder radius='${polerad}' length='${polelen}'/>
     </geometry>
-    <origin rpy='0 0 0' xyz='-${baselen/2} 0 ${basethick/2}'/>
-    <material name='blue'></material>
+    <origin rpy='0 0 0' xyz='0 0 ${polelen/2}'/>
+    <material name='green'></material>
   </visual>
   <collision>
     <geometry>
-      <box size='0.3 ${baselen} 0.05'/>
+      <cylinder radius='${polerad}' length='${polelen}'/>
     </geometry>
-    <origin rpy='0 0 0' xyz='-${baselen/2} 0 ${basethick/2}'/>
+    <origin rpy='0 0 0' xyz='0 0 -${polelen/2}'/>
   </collision>
 </link>
-<!-- Link for pismatic joint -->
-<xacro:sh_link name='1' z='-${basethick/2}' material='grey'>
-  <box size='${sh1len} ${sh1len} ${basethick}'/>
+<!-- Plate connecting base to prismatic joints -->
+<xacro:sh_link name='1' x='${basepllen/2-polerad*1.1}' z='${basethick/2}' material='blue'>
+  <box size='${basepllen} 0.3 ${basethick}'/>
 </xacro:sh_link>
 <!-- Link for pismatic joint -->
@@ -65,76 +97,109 @@
   <box size='${sh1len} ${sh1len} ${basethick}'/>
 </xacro:sh_link>
+<!-- Link for pismatic joint -->
+<xacro:sh_link name='3' z='-${basethick/2}' material='grey'>
+  <box size='${sh1len} ${sh1len} ${basethick}'/>
+</xacro:sh_link>
 <!-- Motor for first revolute joint -->
-<xacro:sh_link name='3' z='-${mot1len/2}' material='black'>
+<xacro:sh_link name='4' z='-${mot1len/2}' material='black'>
   <cylinder radius='${mot1rad}' length='${mot1len}'/>
 </xacro:sh_link>
 <!-- Links for second revolute joint -->
-<xacro:sh_link name='4' z='-${basethick/2}' y='-${conn2len/2-mot1rad*1.1}'>
+<xacro:sh_link name='5' z='-${basethick/2}' y='-${conn2len/2-mot1rad*1.1}'>
   <box size='0.3 ${conn2len} ${basethick}'/>
 </xacro:sh_link>
-<xacro:sh_link name='5' z='-${conn3len/2}'>
+<xacro:sh_link name='6' z='-${conn3len/2}'>
   <box size='0.3 ${basethick} ${conn3len}'/>
 </xacro:sh_link>
 <!-- Motor for second revolute joint -->
-<xacro:sh_link name='6' roll='${pi/2}' y='-${mot2len/2}' material='black'>
+<xacro:sh_link name='7' roll='${pi/2}' y='-${mot2len/2}' material='black'>
   <cylinder radius='${mot2rad}' length='${mot2len}'/>
 </xacro:sh_link>
 <!-- Third prismatic connection -->
-<xacro:sh_link name='7' y='${basethick/2}' material='grey'>
+<xacro:sh_link name='8' y='${basethick/2}' material='grey'>
   <box size='${prism3len} ${basethick} ${prism3len}'/>
 </xacro:sh_link>
-<xacro:sh_link name='8' z='-${conn4len/2-mot2rad*1.1}' y='${basethick/2}'>
+<xacro:sh_link name='9' z='-${conn4len/2-mot2rad*1.1}' y='${basethick/2}'>
   <box size='0.3 ${basethick} ${conn4len}'/>
 </xacro:sh_link>
 <!-- Motor for third revolute joint -->
-<xacro:sh_link name='9' z='${mot3len/2}' material='black'>
+<xacro:sh_link name='10' z='${mot3len/2}' material='black'>
   <cylinder radius='${mot3rad}' length='${mot3len}'/>
 </xacro:sh_link>
 <!-- Interface to human shoulder -->
-<xacro:sh_link name='10' y='${shintrad}' z='${shintthick/2}' material='grey'>
+<xacro:sh_link name='11' z='${shintthick/2}' material='grey'>
   <cylinder radius='${shintrad}' length='${shintthick}'/>
 </xacro:sh_link>
-<!-- <xacro:sh_link name='8'></xacro:sh_link> -->
-<!-- <xacro:sh_link name='9'></xacro:sh_link> -->
-<!-- <xacro:sh_link name='11'></xacro:sh_link> -->
 <!-- First prismatic passive joint -->
-<joint name='base_to_shoulder1' type='prismatic'>
+<joint name='base_to_shoulder1' type='fixed'>
   <parent link='base_link'/>
   <child link='shoulder1'/>
-  <origin rpy='0 0 0' xyz='-${sh1len/2} 0 0'/>
-  <limit effort='50' lower='-0.1' upper='0.1' velocity='5.0'/>
-  <axis xyz='0 1 0'/>
+  <origin rpy='0 0 -${pi/12}' xyz='0 0 ${polelen}'/>
 </joint>
+<!-- Base connecting plate to prismatic joint -->
+<xacro:sh_joint parent='1' child='2' type='prismatic' x='${basepllen-polerad*1.1-sh1len/2}' axisy='1'>
+</xacro:sh_joint>
 <!-- Second prismatic passive joint -->
-<xacro:sh_joint parent='1' child='2' type='prismatic' z='-${basethick}' axisx='1'>
+<xacro:sh_joint parent='2' child='3' type='prismatic' z='-${basethick}' axisx='1'>
 </xacro:sh_joint>
 <!-- Fixed joint between prismatic and revolute joint -->
-<xacro:sh_joint parent='2' child='3' z='-${basethick}'>
+<xacro:sh_joint parent='3' child='4' z='-${basethick}'>
 </xacro:sh_joint>
 <!-- First revolute active joint -->
-<xacro:sh_joint parent='3' child='4' type='continuous' z='-${mot1len}' axisz='1'>
-</xacro:sh_joint>
-<xacro:sh_joint parent='4' child='5' y='-${conn2len-mot1rad*1.1+basethick/2}'>
-</xacro:sh_joint>
-<xacro:sh_joint parent='5' child='6' y='-${basethick/2}' z='-${conn3len-mot2rad*1.1}'>
+<xacro:sh_joint parent='4' child='5' type='continuous' z='-${mot1len}' axisz='1'>
+</xacro:sh_joint>
+<xacro:sh_joint parent='5' child='6' y='-${conn2len-mot1rad*1.1+basethick/2}'>
+</xacro:sh_joint>
+<xacro:sh_joint parent='6' child='7' y='-${basethick/2}' z='-${conn3len-mot2rad*1.1}'>
 </xacro:sh_joint>
 <!-- Second revolute active joint -->
-<xacro:sh_joint parent='6' child='7' type='continuous' y='${basethick}' axisy='1'>
+<xacro:sh_joint parent='7' child='8' type='continuous' y='${basethick}' axisy='1'>
 </xacro:sh_joint>
 <!-- Third prismatic passive joint -->
-<xacro:sh_joint parent='7' child='8' type='prismatic' y='${basethick}' axisz='1'>
-</xacro:sh_joint>
-<xacro:sh_joint parent='8' child='9' z='-${conn4len-mot2rad*1.1}' y='-${mot3rad}'>
+<xacro:sh_joint parent='8' child='9' type='prismatic' y='${basethick}' axisz='1'>
+</xacro:sh_joint>
+<xacro:sh_joint parent='9' child='10' z='-${conn4len-mot2rad*1.1}' y='-${mot3rad}'>
 </xacro:sh_joint>
 <!-- Shoulder interface fixed connection -->
-<xacro:sh_joint parent='8' child='10' z='-${conn4len-mot2rad*1.1}' y='${basethick/2}'>
-</xacro:sh_joint>
-<!-- <xacro:sh_joint parent='6' child='7' type='continuous'></xacro:sh_joint> -->
-<!-- <xacro:sh_joint parent='7' child='8'></xacro:sh_joint> -->
-<!-- <xacro:sh_joint parent='8' child='9' type='prismatic'></xacro:sh_joint> -->
-<!-- <xacro:sh_joint parent='9' child='10' type='continuous'></xacro:sh_joint> -->
-<!-- <xacro:sh_joint parent='10' child='11'></xacro:sh_joint> -->
-<!-- [> Elbow links and joints <] -->
-<!-- <xacro:el_link name='1'></xacro:el_link> -->
+<xacro:sh_joint parent='9' child='11' z='-${conn4len-mot2rad*1.1}' y='${basethick+shintrad}'>
+</xacro:sh_joint>
+<!-- Elbow links and joints -->
+<!-- Shoulder to elbow two reflected links -->
+<xacro:el_link name='1' z='-${elcon1len/2}' x='${shintrad-elcon1thick}' reflectx='-1'>
+  <box size='${elcon1thick} ${elcon1width} ${elcon1len}'/>
+</xacro:el_link>
+<xacro:el_link name='2' z='-${elcon1len/2}' x='${shintrad-elcon1thick}' reflectx='1'>
+  <box size='${elcon1thick} ${elcon1width} ${elcon1len}'/>
+</xacro:el_link>
+<!-- Elbow to forearm reflected links -->
+<xacro:el_link name='3' z='-${elcon2len/2*0.9}' x='${shintrad-elcon1thick-elcon2thick}'
+  reflectx='-1'>
+  <box size='${elcon2thick} ${elcon2width} ${elcon2len}'/>
+</xacro:el_link>
+<xacro:el_link name='4' z='-${elcon2len/2*0.9}' x='${shintrad-elcon1thick-elcon2thick}'
+  reflectx='1'>
+  <box size='${elcon2thick} ${elcon2width} ${elcon2len}'/>
+</xacro:el_link>
+<!-- Motor for fourth revolute joint -->
+<xacro:el_link name='5' pitch='${pi/2}' x='${mot4len/2}' material='black'>
+  <cylinder radius='${mot4rad}' length='${mot4len}'/>
+</xacro:el_link>
+<!-- Fourth prismatic connections -->
+<xacro:el_link name='6' x='${shintrad-elcon1thick-elcon2thick/2+prism4thick/2}'
+  reflectx='-1' material='grey'>
+  <box size='${prism4thick} ${prism4width} ${prism4len}'/>
+</xacro:el_link>
+<xacro:el_link name='7' x='${shintrad-elcon1thick-elcon2thick/2+prism4thick/2}'
+  reflectx='1' material='grey'>
+  <box size='${prism4thick} ${prism4width} ${prism4len}'/>
+</xacro:el_link>
+<!-- Interface to human elbow -->
+<xacro:el_link name='8' z='-${elintthick/2}' material='grey'>
+  <cylinder radius='${elintrad}' length='${elintthick}'/>
+</xacro:el_link>
+<!-- Motor for fifth revolute joint -->
+<xacro:el_link name='9' material='black'>
+  <cylinder radius='${mot5rad}' length='${mot5len}'/>
+</xacro:el_link>
 <!-- <xacro:el_link name='2'></xacro:el_link> -->
 <!-- <xacro:el_link name='3'></xacro:el_link> -->
@@ -142,9 +207,32 @@
 <!-- <xacro:el_link name='4'></xacro:el_link> -->
 <!-- <xacro:el_link name='5'></xacro:el_link> -->
-<!-- <joint name='sh11_el1' type='continuous'> -->
-  <!-- <parent link='shoulder11'/> -->
-  <!-- <child link='elbow1'/> -->
-  <!-- <origin rpy='0 0 0' xyz='0 0 0'/> -->
-<!-- </joint> -->
+<!-- Shoulder to elbow revolute joint -->
+<xacro:el_cust_joint name='sh11_to_el1_rot' type='continuous'
+  parent='shoulder11' child='elbow1' axisz='1'>
+</xacro:el_cust_joint>
+<xacro:el_cust_refl_joint name='sh11_to_el2_rot' type='continuous' mimic='sh11_to_el1_rot'
+  parent='shoulder11' child='elbow2' axisz='1'>
+</xacro:el_cust_refl_joint>
+<!-- Elbow to forearm revolute joint -->
+<xacro:el_joint parent='1' child='3' type='continuous' z='-${elcon1len*0.9}' axisx='1'>
+</xacro:el_joint>
+<xacro:el_refl_joint parent='2' child='4' type='continuous' mimic='el1_el3'
+  z='-${elcon1len*0.9}' axisx='1'>
+</xacro:el_refl_joint>
+<!-- Fourth motor fixed connection -->
+<xacro:el_joint parent='1' child='5' x='${shintrad-elcon1thick/2}' z='-${elcon1len*0.9}'>
+</xacro:el_joint>
+<!-- Fourth prismatic joint -->
+<xacro:el_joint parent='3' child='6' type='prismatic' z='-${elcon2len*0.9}' axisz='1'>
+</xacro:el_joint>
+<xacro:el_refl_joint parent='4' child='7' type='prismatic' z='-${elcon2len*0.9}' axisz='1'
+  mimic='el3_el6'>
+</xacro:el_refl_joint>
+<!-- Elbow interface fixed connection -->
+<xacro:el_joint parent='6' child='8' z='-${prism4len/2}'>
+</xacro:el_joint>
+<!-- Fifth motor fixed connection -->
+<xacro:el_joint parent='8' child='9' x='${elintrad+mot5rad/2}' z='0'>
+</xacro:el_joint>
 <!-- <xacro:el_joint parent='1' child='2'></xacro:el_joint> -->
 <!-- <xacro:el_joint parent='2' child='3' type='prismatic'></xacro:el_joint> -->
