Commit message: UpperExtremity Model proper z-axis orientation in Rviz, add prismatic joint.

File: urdf/UpperExtremity/upper_extremity.urdf (robot description, URDF)
Before this commit: robot UpperExtremityModel, 40 links, 39 joints
Links:
- removed link base_link
- added link ground
Joints:
- joint ground_joint: origin xyz=0 0 0 rpy=0 -0 0 -> xyz=0 0 0 rpy=1.570796327 -0 0; parent base_link -> ground
