Commit message: Partial RehabConcept URDF to passive prismatic wrist joint.

File: urdf/RehabConcept/rehab_concept.urdf (robot description, URDF)
Before this commit: robot RehabConcept, 7 links, 6 joints
Links:
- added link Act2_link, mass 1.0; visual mesh filename=file:///home/tomislav/ros/catkin_tutor/src/rehab/urdf/Rehab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 scale=0.2379111349582672 0.2379111349582672 0.2379111349582672
- added link Act3_link, mass 1.0; visual mesh filename=file:///home/tomislav/ros/catkin_tutor/src/rehab/urdf/Rehab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 scale=0.2379111349582672 0.2379111349582672 0.2379111349582672
- added link Act4_link, mass 1.0; visual mesh filename=file:///home/tomislav/ros/catkin_tutor/src/rehab/urdf/Rehab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 scale=1 1 1
- added link Act5_link, mass 1.0; visual mesh filename=file:///home/tomislav/ros/catkin_tutor/src/rehab/urdf/Rehab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 scale=1 1 1
- added link ElbowLink1_link, mass 1.0; visual mesh filename=file:///home/tomislav/ros/catkin_tutor/src/rehab/urdf/Rehab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 scale=1 1 1
- added link ElbowWristLink_link, mass 1.0; visual mesh filename=file:///home/tomislav/ros/catkin_tutor/src/rehab/urdf/Rehab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 scale=1 1 1
- added link Prism2Base_link, mass 1.0; visual mesh filename=file:///home/tomislav/ros/catkin_tutor/src/rehab/urdf/Rehab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 scale=1 1 1
- added link Prism3Base_link, mass 1.0; visual mesh filename=file:///home/tomislav/ros/catkin_tutor/src/rehab/urdf/Rehab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 scale=1 1 1
- added link Prism3MidSlider_link, mass 1.0; visual mesh filename=file:///home/tomislav/ros/catkin_tutor/src/rehab/urdf/Rehab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 scale=1 1 1
- added link ShoulderInterface_link, mass 1.0; visual mesh filename=file:///home/tomislav/ros/catkin_tutor/src/rehab/urdf/Rehab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 scale=0.824152946472168 0.824152946472168 0.8999999761581421
- added link ShoulderLink2_link, mass 1.0; visual mesh filename=file:///home/tomislav/ros/catkin_tutor/src/rehab/urdf/Rehab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 scale=1 1 1
- added link ShoulderLink3_link, mass 1.0; visual mesh filename=file:///home/tomislav/ros/catkin_tutor/src/rehab/urdf/Rehab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 scale=1 1 1
Joints:
- added joint Act2_joint: type fixed, parent ShoulderLink2_link, child Act2_link, origin xyz=-0.06065359711647034 0 0 rpy=0 -0 0, axis 0 0 1, limit lower=1.0 upper=1.0 effort=100.0 velocity=1.0
- added joint Act3_joint: type fixed, parent ShoulderLink2_link, child Act3_link, origin xyz=0 -0.15047705173492432 0.03126099705696106 rpy=0 -0 0, axis 0 0 1, limit lower=1.0 upper=1.0 effort=100.0 velocity=1.0
- added joint Act4_joint: type fixed, parent ShoulderLink3_link, child Act4_link, origin xyz=0 -0.16287004947662354 0.005409032106399536 rpy=0 -0 0, axis 0 0 1, limit lower=1.0 upper=1.0 effort=100.0 velocity=1.0
- added joint Act5_joint: type fixed, parent ElbowWristLink_link, child Act5_link, origin xyz=0 0 0.01441279798746109 rpy=0 -0 0, axis 0 0 1, limit lower=1.0 upper=1.0 effort=100.0 velocity=1.0
- added joint ElbowLink1_joint: type revolute, parent ShoulderLink3_link, child ElbowLink1_link, origin xyz=0 -0.17770802974700928 -0.09135209769010544 rpy=0 -0 0, axis 0 1 0, limit lower=-2.0943951023931953 upper=2.0943951023931953 effort=100.0 velocity=1.0
- added joint ElbowWristLink_joint: type revolute, parent ElbowLink1_link, child ElbowWristLink_link, origin xyz=-2.7418136596679688e-06 -0.12219798564910889 0.055660001933574677 rpy=0 -0 0, axis 0 0 1, limit lower=-0.17453292519943295 upper=3.141592653589793 effort=100.0 velocity=1.0
- added joint Prism2Base_joint: type revolute, parent ShoulderLink2_link, child Prism2Base_link, origin xyz=0 -0.15047705173492432 -0.036590397357940674 rpy=0 -0 0, axis 0 0 1, limit lower=-1.0471975511965976 upper=3.141592653589793 effort=100.0 velocity=1.0
- added joint Prism3Base_joint: type fixed, parent ElbowWristLink_link, child Prism3Base_link, origin xyz=-0.06398391723632812 -0.16407698392868042 -0.02864900231361389 rpy=0 -0 0, axis 0 0 1, limit lower=1.0 upper=1.0 effort=100.0 velocity=1.0
- added joint Prism3MidSlider_joint: type prismatic, parent Prism3Base_link, child Prism3MidSlider_link, origin xyz=0 -0.0016984939575195312 0 rpy=0 -0 0, axis 0 1 0, limit lower=-0.05000000074505806 upper=0.05000000074505806 effort=100.0 velocity=1.0
- added joint ShoulderInterface_joint: type fixed, parent ElbowLink1_link, child ShoulderInterface_link, origin xyz=0 0 0 rpy=0 -0 0, axis 0 0 1, limit lower=1.0 upper=1.0 effort=100.0 velocity=1.0
- added joint ShoulderLink2_joint: type revolute, parent ShoulderLink1_link, child ShoulderLink2_link, origin xyz=0 0.01687788963317871 0.14730499684810638 rpy=0 -0 0, axis 1 0 0, limit lower=-2.0943951023931953 upper=0.5235987755982988 effort=100.0 velocity=1.0
- added joint ShoulderLink3_joint: type prismatic, parent Prism2Base_link, child ShoulderLink3_link, origin xyz=0 0.005881309509277344 0 rpy=0 -0 0, axis 0 1 0, limit lower=-0.10000000149011612 upper=0.30000001192092896 effort=100.0 velocity=1.0
- joint Prism1Connector_joint: limit lower=-90.0 upper=90.0 effort=100.0 velocity=1.0 -> lower=-0.05000000074505806 upper=0.05000000074505806 effort=100.0 velocity=1.0
- joint Prism1MidSlider_joint: axis 0 1 0 -> 0 0 1; limit lower=-90.0 upper=90.0 effort=100.0 velocity=1.0 -> lower=-0.05000000074505806 upper=0.05000000074505806 effort=100.0 velocity=1.0
- joint ShoulderLink1_joint: axis 0 0 1 -> 0 1 0; limit lower=-1.5707963267948966 upper=1.5707963267948966 effort=100.0 velocity=1.0 -> lower=-2.0943951023931953 upper=1.5707963267948966 effort=100.0 velocity=1.0

Commit message: Add RehabConcept links and joints to HandInterfaceBase.

File: urdf/RehabConcept/rehab_concept.urdf (robot description, URDF)
Before this commit: robot RehabConcept, 19 links, 18 joints
Links:
- added link Act6_link, mass 1.0; visual mesh filename=file:///home/tomislav/ros/catkin_tutor/src/rehab/urdf/Rehab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 scale=1 1 1
- added link Act7_link, mass 1.0; visual mesh filename=file:///home/tomislav/ros/catkin_tutor/src/rehab/urdf/Rehab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 scale=1 1 1
- added link Act8_link, mass 1.0; visual mesh filename=file:///home/tomislav/ros/catkin_tutor/src/rehab/urdf/Rehab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 scale=1.04426908493042 1.04426908493042 1.04426908493042
- added link ElasticHingePart1_link, mass 1.0; visual mesh filename=file:///home/tomislav/ros/catkin_tutor/src/rehab/urdf/Rehab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 scale=1 1 1
- added link ElasticHingePart2_link, mass 1.0; visual mesh filename=file:///home/tomislav/ros/catkin_tutor/src/rehab/urdf/Rehab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 scale=1 1 1
- added link ElbowInterface_link, mass 1.0; visual mesh filename=file:///home/tomislav/ros/catkin_tutor/src/rehab/urdf/Rehab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 scale=1 1 1
- added link HandInterfaceBase_link, mass 1.0; visual mesh filename=file:///home/tomislav/ros/catkin_tutor/src/rehab/urdf/Rehab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 scale=1 1 1
- added link Prism4Base_link, mass 1.0; visual mesh filename=file:///home/tomislav/ros/catkin_tutor/src/rehab/urdf/Rehab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 scale=1 1 1
- added link Prism4MidSlider_link, mass 1.0; visual mesh filename=file:///home/tomislav/ros/catkin_tutor/src/rehab/urdf/Rehab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 scale=1 1 1
- added link WristLink1_link, mass 1.0; visual mesh filename=file:///home/tomislav/ros/catkin_tutor/src/rehab/urdf/Rehab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 scale=1 1 1
- added link WristLink2_link, mass 1.0; visual mesh filename=file:///home/tomislav/ros/catkin_tutor/src/rehab/urdf/Rehab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 scale=1 1 1
- added link WristLink3_link, mass 1.0; visual mesh filename=file:///home/tomislav/ros/catkin_tutor/src/rehab/urdf/Rehab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 scale=1 1 1
- added link WristRail1_link, mass 1.0; visual mesh filename=file:///home/tomislav/ros/catkin_tutor/src/rehab/urdf/Rehab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 scale=0.9575729966163635 0.9575729966163635 0.9575729966163635
- added link WristRail2_link, mass 1.0; visual mesh filename=file:///home/tomislav/ros/catkin_tutor/src/rehab/urdf/Rehab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 scale=0.9575730562210083 0.9575730562210083 0.9575730562210083
- added link WristSlider1_link, mass 1.0; visual mesh filename=file:///home/tomislav/ros/catkin_tutor/src/rehab/urdf/Rehab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 scale=1 1 1
- added link WristSlider2_link, mass 1.0; visual mesh filename=file:///home/tomislav/ros/catkin_tutor/src/rehab/urdf/Rehab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 scale=1 1 1
Joints:
- added joint Act6_joint: type fixed, parent WristSlider2_link, child Act6_link, origin xyz=-0.056956589221954346 -0.0025862455368041992 0 rpy=0 -0 0, axis 0 0 1, limit lower=1.0 upper=1.0 effort=100.0 velocity=1.0
- added joint Act7_joint: type fixed, parent WristLink2_link, child Act7_link, origin xyz=-0.0030038952827453613 0 0 rpy=0 -0 0, axis 0 0 1, limit lower=1.0 upper=1.0 effort=100.0 velocity=1.0
- added joint Act8_joint: type fixed, parent ElasticHingePart1_link, child Act8_link, origin xyz=0 0 0.010814502835273743 rpy=0 -0 0, axis 0 0 1, limit lower=1.0 upper=1.0 effort=100.0 velocity=1.0
- added joint ElasticHingePart1_joint: type revolute, parent WristLink2_link, child ElasticHingePart1_link, origin xyz=0.06232398748397827 -0.0008130073547363281 0.08572039008140564 rpy=0 -0 0, axis 0 0 1, limit lower=-0.5235987755982988 upper=1.3962634015954636 effort=100.0 velocity=1.0
- added joint ElasticHingePart2_joint: type revolute, parent ElasticHingePart1_link, child ElasticHingePart2_link, origin xyz=0 -0.03731536865234375 0 rpy=0 -0 0, axis 0 0 1, limit lower=-0.5235987755982988 upper=0.5235987755982988 effort=100.0 velocity=1.0
- added joint ElbowInterface_joint: type fixed, parent WristLink1_link, child ElbowInterface_link, origin xyz=0 0 0 rpy=0 -0 0, axis 0 0 1, limit lower=1.0 upper=1.0 effort=100.0 velocity=1.0
- added joint HandInterfaceBase_joint: type fixed, parent WristLink3_link, child HandInterfaceBase_link, origin xyz=-0.012044697999954224 -0.004274606704711914 -0.10489299893379211 rpy=0 -0 0, axis 0 0 1, limit lower=1.0 upper=1.0 effort=100.0 velocity=1.0
- added joint Prism4Base_joint: type fixed, parent ElasticHingePart2_link, child Prism4Base_link, origin xyz=0 -0.03698563575744629 0 rpy=0 -0 0, axis 0 0 1, limit lower=1.0 upper=1.0 effort=100.0 velocity=1.0
- added joint Prism4MidSlider_joint: type revolute, parent Prism4Base_link, child Prism4MidSlider_link, origin xyz=0 -0.009239494800567627 0 rpy=0 -0 0, axis 0 1 0, limit lower=-0.00034906584259663615 upper=0.00034906584259663615 effort=100.0 velocity=1.0
- added joint WristLink1_joint: type revolute, parent WristSlider2_link, child WristLink1_link, origin xyz=0 -0.01816105842590332 0 rpy=0 -0 0, axis 0 1 0, limit lower=-1.5707963267948966 upper=1.5707963267948966 effort=100.0 velocity=1.0
- added joint WristLink2_joint: type revolute, parent WristLink1_link, child WristLink2_link, origin xyz=-0.055825501680374146 -0.10307097434997559 0.007611200213432312 rpy=0 -0 0, axis 1 0 0, limit lower=-1.5707963267948966 upper=1.5707963267948966 effort=100.0 velocity=1.0
- added joint WristLink3_joint: type fixed, parent Prism4MidSlider_link, child WristLink3_link, origin xyz=0.012020885944366455 -5.960464477539063e-08 0 rpy=0 -0 0, axis 0 0 1, limit lower=1.0 upper=1.0 effort=100.0 velocity=1.0
- added joint WristRail1_joint: type fixed, parent WristLink1_link, child WristRail1_link, origin xyz=0 0.015488743782043457 0 rpy=0 -0 0, axis 0 0 1, limit lower=1.0 upper=1.0 effort=100.0 velocity=1.0
- added joint WristRail2_joint: type fixed, parent WristLink1_link, child WristRail2_link, origin xyz=0 -0.015488862991333008 0 rpy=0 -0 0, axis 0 0 1, limit lower=1.0 upper=1.0 effort=100.0 velocity=1.0
- added joint WristSlider1_joint: type fixed, parent Prism3MidSlider_link, child WristSlider1_link, origin xyz=0.09463348984718323 -0.017802953720092773 0 rpy=0 -0 0, axis 0 0 1, limit lower=1.0 upper=1.0 effort=100.0 velocity=1.0
- added joint WristSlider2_joint: type fixed, parent Prism3MidSlider_link, child WristSlider2_link, origin xyz=0.09463348984718323 0.018518686294555664 0 rpy=0 -0 0, axis 0 0 1, limit lower=1.0 upper=1.0 effort=100.0 velocity=1.0

Commit message: Finished DH coordinate systems, render RehabConcept.

File: urdf/RehabConcept/rehab_concept.urdf (robot description, URDF)
Before this commit: robot RehabConcept, 35 links, 34 joints
Links:
- added link HandInterfaceBack_link, mass 1.0; visual mesh filename=file:///home/tomislav/ros/catkin_tutor/src/rehab/urdf/Rehab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 scale=1 1 1
- added link HandInterfaceIndex_link, mass 1.0; visual mesh filename=file:///home/tomislav/ros/catkin_tutor/src/rehab/urdf/Rehab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 scale=1 1 1
- added link HandInterfaceLittle_link, mass 1.0; visual mesh filename=file:///home/tomislav/ros/catkin_tutor/src/rehab/urdf/Rehab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 scale=1 1 1
- added link HandInterfaceMiddle_link, mass 1.0; visual mesh filename=file:///home/tomislav/ros/catkin_tutor/src/rehab/urdf/Rehab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 scale=1 1 1
- added link HandInterfaceRing_link, mass 1.0; visual mesh filename=file:///home/tomislav/ros/catkin_tutor/src/rehab/urdf/Rehab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 scale=1 1 1
- added link SpringIndex_link, mass 1.0; visual mesh filename=file:///home/tomislav/ros/catkin_tutor/src/rehab/urdf/Rehab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 scale=1 1 1
- added link SpringLittle_link, mass 1.0; visual mesh filename=file:///home/tomislav/ros/catkin_tutor/src/rehab/urdf/Rehab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 scale=1 1 1
- added link SpringMiddle_link, mass 1.0; visual mesh filename=file:///home/tomislav/ros/catkin_tutor/src/rehab/urdf/Rehab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 scale=1 1 1
- added link SpringRing_link, mass 1.0; visual mesh filename=file:///home/tomislav/ros/catkin_tutor/src/rehab/urdf/Rehab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 scale=1 1 1
- added link SpringsBack_link, mass 1.0; visual mesh filename=file:///home/tomislav/ros/catkin_tutor/src/rehab/urdf/Rehab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 scale=1 1 1
Joints:
- added joint HandInterfaceBack_joint: type fixed, parent SpringsBack_link, child HandInterfaceBack_link, origin xyz=0.01538550853729248 -0.012692689895629883 0 rpy=0 -0 0, axis 0 0 1, limit lower=1.0 upper=1.0 effort=100.0 velocity=1.0
- added joint HandInterfaceIndex_joint: type fixed, parent SpringIndex_link, child HandInterfaceIndex_link, origin xyz=0 -0.010886132717132568 0 rpy=0 -0 0, axis 0 0 1, limit lower=1.0 upper=1.0 effort=100.0 velocity=1.0
- added joint HandInterfaceLittle_joint: type fixed, parent SpringLittle_link, child HandInterfaceLittle_link, origin xyz=0 -0.01087808609008789 0 rpy=0 -0 0, axis 0 0 1, limit lower=1.0 upper=1.0 effort=100.0 velocity=1.0
- added joint HandInterfaceMiddle_joint: type fixed, parent SpringMiddle_link, child HandInterfaceMiddle_link, origin xyz=0 -0.010810434818267822 0 rpy=0 -0 0, axis 0 0 1, limit lower=1.0 upper=1.0 effort=100.0 velocity=1.0
- added joint HandInterfaceRing_joint: type fixed, parent SpringRing_link, child HandInterfaceRing_link, origin xyz=0 -0.010808050632476807 0 rpy=0 -0 0, axis 0 0 1, limit lower=1.0 upper=1.0 effort=100.0 velocity=1.0
- added joint SpringIndex_joint: type prismatic, parent HandInterfaceBase_link, child SpringIndex_link, origin xyz=0.019673287868499756 -0.0037446022033691406 0 rpy=0 -0 0, axis 0 1 0, limit lower=0.0 upper=0.009999999776482582 effort=100.0 velocity=1.0
- added joint SpringLittle_joint: type prismatic, parent HandInterfaceBase_link, child SpringLittle_link, origin xyz=-0.025188297033309937 -0.0017123222351074219 0 rpy=0 -0 0, axis 0 1 0, limit lower=0.0 upper=0.009999999776482582 effort=100.0 velocity=1.0
- added joint SpringMiddle_joint: type prismatic, parent HandInterfaceBase_link, child SpringMiddle_link, origin xyz=0.003566145896911621 -0.0030896663665771484 0 rpy=0 -0 0, axis 0 1 0, limit lower=0.0 upper=0.009999999776482582 effort=100.0 velocity=1.0
- added joint SpringRing_joint: type prismatic, parent HandInterfaceBase_link, child SpringRing_link, origin xyz=-0.011842310428619385 -0.002404451370239258 0 rpy=0 -0 0, axis 0 1 0, limit lower=0.0 upper=0.009999999776482582 effort=100.0 velocity=1.0
- added joint SpringsBack_joint: type prismatic, parent HandInterfaceBase_link, child SpringsBack_link, origin xyz=-0.01538550853729248 0.0192795991897583 0 rpy=0 -0 0, axis 0 1 0, limit lower=-0.009999999776482582 upper=0.0 effort=100.0 velocity=1.0
- joint HandInterfaceBase_joint: origin xyz=-0.012044697999954224 -0.004274606704711914 -0.10489299893379211 rpy=0 -0 0 -> xyz=-0.01126149296760559 -0.004274606704711914 -0.10489299893379211 rpy=0 -0 0
- joint Prism4MidSlider_joint: limit lower=-0.00034906584259663615 upper=0.00034906584259663615 effort=100.0 velocity=1.0 -> lower=-0.02500000037252903 upper=0.02500000037252903 effort=100.0 velocity=1.0; type revolute -> prismatic
