Commit message: Fix ForearmRehabIKFast joint constraints and visual render.

File: models/RehabilitationDeviceForearmHand/ForearmRehabIKFast/model.urdf (robot description, URDF)
Before this commit: robot ForearmRehabIKFast, 11 links, 10 joints
Joints:
- joint ElbowWristLink_joint: limit lower=-1.5707963267948966 upper=0.0 effort=0.0 velocity=0.0 -> lower=-2.2689280275926285 upper=0.0 effort=0.0 velocity=0.0
- joint HandLink_joint: limit lower=-1.0471975511965976 upper=0.5235987755982988 effort=0.0 velocity=0.0 -> lower=-0.4363323129985824 upper=0.17453292519943295 effort=0.0 velocity=0.0
- joint WristLink1_joint: limit lower=-1.9198621771937625 upper=1.9198621771937625 effort=0.0 velocity=0.0 -> lower=-1.5707963267948966 upper=1.5707963267948966 effort=0.0 velocity=0.0
- joint WristLink2_joint: limit lower=-0.9599310885968813 upper=2.0943951023931953 effort=0.0 velocity=0.0 -> lower=-0.9599310885968813 upper=1.2217304763960306 effort=0.0 velocity=0.0
