Commit message: Add dependent joints for hadn and finger by finger, DH parameters in jupyter notebook and R + visualization, fix MCP_AA and MCP_FE joint sequence, add index_tf_publisher for grid motion.

File: urdf/Hand9DOF/hand9dof.urdf (robot description, URDF)
Before this commit: robot Hand9DOF, 26 links, 25 joints
Links:
- link IndexMCP_AA: geometry visual mesh filename=package://rehab/models/RehabilitationDeviceHand/Hand9DOF/me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 scale=1.0 1.0 1.0
- link IndexMCP_FE: geometry 
- link LittleMCP_AA: geometry visual mesh filename=package://rehab/models/RehabilitationDeviceHand/Hand9DOF/me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 scale=1.0 1.0 1.0
- link LittleMCP_FE: geometry 
- link MiddleMCP_AA: geometry visual mesh filename=package://rehab/models/RehabilitationDeviceHand/Hand9DOF/me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 scale=1.0 1.0 1.0
- link MiddleMCP_FE: geometry 
- link RingMCP_AA: geometry visual mesh filename=package://rehab/models/RehabilitationDeviceHand/Hand9DOF/me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 scale=1.0 1.0 1.0
- link RingMCP_FE: geometry 
Joints:
- joint IndexCMC_joint: axis 0.973  0.124 -0.194 -> 0.988 0.153 0.008
- joint IndexDIP_joint: axis 0.997    0.07299 -0.026 -> 0.988 0.153 0.008
- joint IndexMCP_AA_joint: axis -0.058  0.086  0.995 -> -0.03     0.14099  0.99; origin xyz=0.00912 -0.06174  0.01116 rpy=0 0 0 -> xyz=0 0 0 rpy=0 0 0; parent IndexCMC -> IndexMCP_FE
- joint IndexMCP_FE_joint: axis 0.999 0.046 0.022 -> 0.988 0.153 0.008; origin xyz=0 0 0 rpy=0 0 0 -> xyz=0.00912 -0.06174  0.01116 rpy=0 0 0; parent IndexMCP_AA -> IndexCMC
- joint IndexPIP_joint: axis 0.992  0.104 -0.066 -> 0.988 0.153 0.008; parent IndexMCP_FE -> IndexMCP_AA
- joint LittleCMC_joint: axis 0.959 -0.172  0.224 -> 0.898 -0.157  0.412
- joint LittleDIP_joint: axis 0.897 -0.171  0.408 -> 0.898 -0.157  0.412
- joint LittleMCP_AA_joint: axis -0.62   0.021  0.784 -> -0.422 -0.037  0.906; origin xyz=-0.00635 -0.05361 -0.00496 rpy=0 0 0 -> xyz=0 0 0 rpy=0 0 0; parent LittleCMC -> LittleMCP_FE
- joint LittleMCP_FE_joint: axis 0.978 -0.064  0.198 -> 0.898 -0.157  0.412; origin xyz=0 0 0 rpy=0 0 0 -> xyz=-0.00635 -0.05361 -0.00496 rpy=0 0 0; parent LittleMCP_AA -> LittleCMC
- joint LittlePIP_joint: axis 0.894 -0.254  0.368 -> 0.898 -0.157  0.412; parent LittleMCP_FE -> LittleMCP_AA
- joint MiddleCMC_joint: axis 1     0.006 -0.003 -> 0.98  0.052 0.194
- joint MiddleDIP_joint: axis 0.991 0.129 0.029 -> 0.98  0.052 0.194
- joint MiddleMCP_AA_joint: axis 0.059 0.056 0.997 -> -0.198  0.082  0.977; origin xyz=0.00085 -0.06524  0.00901 rpy=0 0 0 -> xyz=0 0 0 rpy=0 0 0; parent MiddleCMC -> MiddleMCP_FE
- joint MiddleMCP_FE_joint: axis 0.997 -0.077  0.026 -> 0.98  0.052 0.194; origin xyz=0 0 0 rpy=0 0 0 -> xyz=0.00085 -0.06524  0.00901 rpy=0 0 0; parent MiddleMCP_AA -> MiddleCMC
- joint MiddlePIP_joint: axis 0.998 0.064 0.026 -> 0.98  0.052 0.194; parent MiddleMCP_FE -> MiddleMCP_AA
- joint RingCMC_joint: axis 0.984 -0.068  0.164 -> 0.949 -0.07   0.309
- joint RingDIP_joint: axis 0.973 -0.039  0.226 -> 0.949 -0.07   0.309
- joint RingMCP_AA_joint: axis -0.386  0.034  0.922 -> -0.305  0.063  0.95; origin xyz=-0.00351 -0.06171  0.00408 rpy=0 0 0 -> xyz=0 0 0 rpy=0 0 0; parent RingCMC -> RingMCP_FE
- joint RingMCP_FE_joint: axis 0.966 -0.083  0.243 -> 0.949 -0.07   0.309; origin xyz=0 0 0 rpy=0 0 0 -> xyz=-0.00351 -0.06171  0.00408 rpy=0 0 0; parent RingMCP_AA -> RingCMC
- joint RingPIP_joint: axis 0.981 -0.063  0.183 -> 0.949 -0.07   0.309; parent RingMCP_FE -> RingMCP_AA
- joint ThumbIP_joint: axis 0.051  0.48  -0.876 -> 0.028  0.407 -0.913
- joint ThumbMCP_joint: axis 0.092  0.204 -0.975 -> 0.028  0.407 -0.913
- joint ThumbTMC_FE_joint: axis 0.049  0.665 -0.745 -> 0.028  0.407 -0.913
